Commit message: first pick&place with errors

File: src/franka_manipulation_env/urdf/system.urdf.xacro (robot description, xacro)
@@ -68,5 +68,5 @@
         <parent link="world"/>
         <child link="camera_link"/>
-        <origin xyz="0.5 0 1.5" rpy="0 1.571 0"/>
+        <origin xyz="0.5 1.0 1.2" rpy="0 0.5 -1.571"/>
     </joint>
     <gazebo reference="camera_link">

Commit message: Ready to test on hardware

File: src/franka_manipulation_env/urdf/system.urdf.xacro (robot description, xacro)
@@ -11,16 +11,16 @@
     <link name="table_link">
         <visual>
-            <origin xyz="0 0 0.375" rpy="0 0 0"/>
+            <origin xyz="0 0 0.375" rpy="0 0 0" />
             <geometry>
-                <box size="1.2 0.8 0.75"/>
+                <box size="1.2 0.8 0.75" />
             </geometry>
             <material name="Wood">
-                <color rgba="0.5 0.3 0.1 1.0"/>
+                <color rgba="0.5 0.3 0.1 1.0" />
             </material>
         </visual>
         <collision>
-            <origin xyz="0 0 0.375" rpy="0 0 0"/>
+            <origin xyz="0 0 0.375" rpy="0 0 0" />
             <geometry>
-                <box size="1.2 0.8 0.75"/>
+                <box size="1.2 0.8 0.75" />
             </geometry>
             <surface>
@@ -35,5 +35,6 @@
                 <friction>
                     <ode>
-                        <mu>100.0</mu> <mu2>100.0</mu2>
+                        <mu>100.0</mu>
+                        <mu2>100.0</mu2>
                     </ode>
                 </friction>
@@ -41,7 +42,7 @@
         </collision>
         <inertial>
-            <mass value="1000.0"/>
-            <origin xyz="0 0 0.375" rpy="0 0 0"/>
-            <inertia ixx="100.0" ixy="0" ixz="0" iyy="100.0" iyz="0" izz="100.0"/>
+            <mass value="1000.0" />
+            <origin xyz="0 0 0.375" rpy="0 0 0" />
+            <inertia ixx="100.0" ixy="0" ixz="0" iyy="100.0" iyz="0" izz="100.0" />
         </inertial>
     </link>
@@ -53,27 +54,33 @@
     <link name="camera_link">
         <visual>
-            <geometry><box size="0.1 0.1 0.05"/></geometry>
-            <material name="Black"><color rgba="0 0 0 1"/></material>
+            <geometry>
+                <box size="0.1 0.1 0.05" />
+            </geometry>
+            <material name="Black">
+                <color rgba="0 0 0 1" />
+            </material>
         </visual>
         <collision>
-            <geometry><box size="0.1 0.1 0.05"/></geometry>
+            <geometry>
+                <box size="0.1 0.1 0.05" />
+            </geometry>
         </collision>
         <inertial>
-            <mass value="0.1"/>
-            <origin xyz="0 0 0" rpy="0 0 0"/>
-            <inertia ixx="0.001" ixy="0" ixz="0" iyy="0.001" iyz="0" izz="0.001"/>
+            <mass value="0.1" />
+            <origin xyz="0 0 0" rpy="0 0 0" />
+            <inertia ixx="0.001" ixy="0" ixz="0" iyy="0.001" iyz="0" izz="0.001" />
         </inertial>
     </link>
     <joint name="world_to_camera" type="fixed">
-        <parent link="world"/>
-        <child link="camera_link"/>
-        <origin xyz="0.5 1.0 1.2" rpy="0 0.5 -1.571"/>
+        <parent link="world" />
+        <child link="camera_link" />
+        <origin xyz="0.5 1.0 1.2" rpy="0 0.5 -1.571" />
     </joint>
     <gazebo reference="camera_link">
-        <sensor name="camera" type="camera">
+        <sensor name="camera" type="rgbd">
             <always_on>1</always_on>
             <update_rate>30</update_rate>
             <visualize>true</visualize>
-            <topic>camera/image_raw</topic>
+            <topic>camera</topic>
             <camera>
                 <horizontal_fov>1.047</horizontal_fov>
@@ -88,9 +95,11 @@
                 </clip>
             </camera>
-            <plugin filename="libignition-gazebo-sensors-system.so" name="ignition::gazebo::systems::Sensors">
+            <plugin filename="libignition-gazebo-sensors-system.so"
+                name="ignition::gazebo::systems::Sensors">
                 <render_engine>ogre2</render_engine>
             </plugin>
         </sensor>
     </gazebo>
-    <xacro:franka_gazebo_control config_file="$(find franka_manipulation_env)/config/fr3_controllers.yaml"/>
+    <xacro:franka_gazebo_control
+        config_file="$(find franka_manipulation_env)/config/fr3_controllers.yaml" />
 </robot>
