Commit message: Simulation Tests

File: src/franka_manipulation_env/urdf/bimanual_custom.urdf.xacro (robot description, xacro)
@@ -8,4 +8,10 @@
     <child link="table" />
   </joint>
+  <!--  _____     _     _       -->
+  <!-- |_   _|_ _| |__ | | ___  -->
+  <!--   | |/ _` | '_ \| |/ _ \ -->
+  <!--   | | (_| | |_) | |  __/ -->
+  <!--   |_|\__,_|_.__/|_|\___| -->
+  <!--                          -->
   <material name="tablematerial">
     <color rgba="0.8 0.8 0.8 1.0" />
@@ -57,12 +63,25 @@
     <origin xyz="0.03 0.48 0.0" />
   </joint>
-  <!-- Configuration Arguments -->
+  <!--  _____                _           ____                                -->
+  <!-- |  ___| __ __ _ _ __ | | ____ _  |  _ \ __ _ _ __ __ _ _ __ ___  ___  -->
+  <!-- | |_ | '__/ _` | '_ \| |/ / _` | | |_) / _` | '__/ _` | '_ ` _ \/ __| -->
+  <!-- |  _|| | | (_| | | | |   < (_| | |  __/ (_| | | | (_| | | | | | \__ \ -->
+  <!-- |_|  |_|  \__,_|_| |_|_|\_\__,_| |_|   \__,_|_|  \__,_|_| |_| |_|___/ -->
+  <!--                                                                       -->
+  <!-- Should an end-effector be mounted at the flange?" -->
   <xacro:arg name="hand" default="true" />
+  <!-- Which end-effector would be mounted at the flange?" -->
   <xacro:arg name="ee_id" default="franka_hand" />
+  <!-- Should self-collision be enabled? -->
   <xacro:arg name="with_sc" default="false" />
+  <!-- Is the robot being controlled with ros2_control?" -->
   <xacro:arg name="ros2_control" default="false" />
+  <!-- Should a fake hardware be used? -->
   <xacro:arg name="use_fake_hardware" default="false" />
+  <!-- Should fake sensors be used? -->
   <xacro:arg name="fake_sensor_commands" default="false" />
+  <!-- Should the robot be spawned in Gazebo?" -->
   <xacro:arg name="gazebo" default="false" />
+  <!-- Should the robot be spawned in Gazebo with effort interfaces?" -->
   <xacro:arg name="gazebo_effort" default="false" />
   <xacro:arg name="multi_arm" default="true" />
@@ -73,5 +92,10 @@
   <xacro:arg name="controller_path"
     default="$(find idra_franka_launch)/config/basic_controllers.yaml" />
-  <!-- Franka Robot 1 -->
+  <!--  _____                _         _  -->
+  <!-- |  ___| __ __ _ _ __ | | ____ _/ | -->
+  <!-- | |_ | '__/ _` | '_ \| |/ / _` | | -->
+  <!-- |  _|| | | (_| | | | |   < (_| | | -->
+  <!-- |_|  |_|  \__,_|_| |_|_|\_\__,_|_| -->
+  <!--                                    -->
   <xacro:franka_robot arm_id="fr3"
     joint_limits="${xacro.load_yaml('$(find franka_description)/robots/fr3/joint_limits.yaml')}"
@@ -93,11 +117,19 @@
     gazebo_effort="$(arg gazebo_effort)"
     rpy_ee="0 0 ${-pi/4}"
-  />
+  >
+  </xacro:franka_robot>
+  <!-- Dimensions taken from technical drawing of Franka plate and custom designed plate, do not
+  touch -->
   <joint name="plate_to_franka1" type="fixed">
     <parent link="robot1_plate" />
     <child link="franka1_fr3_link0" />
-    <origin xyz="0.145 0.107 0.018" rpy="0 0 ${-pi/2}" />
-  </joint>
-  <!-- Franka Robot 2 -->
+    <origin xyz="0.145 0.107 0.018" rpy="0 0 ${pi}" />
+  </joint>
+  <!--  _____                _         ____   -->
+  <!-- |  ___| __ __ _ _ __ | | ____ _|___ \  -->
+  <!-- | |_ | '__/ _` | '_ \| |/ / _` | __) | -->
+  <!-- |  _|| | | (_| | | | |   < (_| |/ __/  -->
+  <!-- |_|  |_|  \__,_|_| |_|_|\_\__,_|_____| -->
+  <!--                                        -->
   <xacro:franka_robot arm_id="fr3"
     joint_limits="${xacro.load_yaml('$(find franka_description)/robots/fr3/joint_limits.yaml')}"
@@ -119,21 +151,28 @@
     gazebo_effort="$(arg gazebo_effort)"
     rpy_ee="0 0 ${-pi/4}"
-  />
+  >
+  </xacro:franka_robot>
+  <!-- Dimensions taken from technical drawing of Franka plate and custom designed plate, do not
+  touch -->
   <joint name="plate_to_franka2" type="fixed">
     <parent link="robot2_plate" />
     <child link="franka2_fr3_link0" />
-    <origin xyz="0.145 0.107 0.018" rpy="0 0 ${-pi/2}" />
-  </joint>
-  <!-- Hardware Interface Spawner -->
-  <xacro:macro name="interface_spawner" params="robot_name">
-    <xacro:macro name="configure_joint" params="joint_name initial_position is_mimic:=false">
+    <origin xyz="0.145 0.107 0.018" rpy="0 0 0" />
+  </joint>
+  <!-- TODO: add if based on ros2_control arg -->
+  <xacro:macro name="interface_spawner" params="robot_name initial_j1">
+    <!-- Joint position, velocity and effort interfaces -->
+    <xacro:macro name="configure_joint" params="joint_name initial_position">
       <joint name="${joint_name}">
-        <xacro:unless value="${is_mimic}">
-          <command_interface name="position" />
-          <command_interface name="velocity" />
-          <xacro:if value="$(eval not gazebo or gazebo_effort)">
-            <command_interface name="effort" />
-          </xacro:if>
-        </xacro:unless>
+        <!--
+          deactivated for gazebo velocity and position interface due to a bug
+          https://github.com/ros-controls/gz_ros2_control/issues/343
+          Command Interfaces -->
+        <command_interface name="position" />
+        <command_interface name="velocity" />
+        <xacro:if value="$(eval not gazebo or gazebo_effort)">
+          <command_interface name="effort" />
+        </xacro:if>
+        <!-- State Interfaces -->
         <state_interface name="position">
           <param name="initial_value">${initial_position}</param>
@@ -150,5 +189,5 @@
       </gpio>
     </xacro:macro>
-    <xacro:configure_joint joint_name="${robot_name}_fr3_joint1" initial_position="0.0" />
+    <xacro:configure_joint joint_name="${robot_name}_fr3_joint1" initial_position="${initial_j1}" />
     <xacro:configure_joint joint_name="${robot_name}_fr3_joint2" initial_position="${-pi/4}" />
     <xacro:configure_joint joint_name="${robot_name}_fr3_joint3" initial_position="0.0" />
@@ -159,11 +198,11 @@
     <xacro:if value="$(eval gazebo and hand)">
       <xacro:configure_joint joint_name="${robot_name}_fr3_finger_joint1" initial_position="0.0" />
-      <xacro:configure_joint joint_name="${robot_name}_fr3_finger_joint2" initial_position="0.0" />
     </xacro:if>
-    <!-- Elbow & Cartesian interfaces -->
+    <!-- Elbow interfaces -->
     <xacro:general_purpose_io prefix="${robot_name}_joint_3_position"
       command_interface="elbow_command" index="0" />
     <xacro:general_purpose_io prefix="${robot_name}_joint_4_sign" command_interface="elbow_command"
       index="1" />
+    <!-- Cartesian position interfaces -->
     <xacro:macro name="loop" params="i">
       <xacro:unless value="${i == 16}">
@@ -174,4 +213,5 @@
     </xacro:macro>
     <xacro:loop i="0" />
+    <!-- Cartesian pose (position + quaternion) interface -->
     <xacro:general_purpose_io prefix="${robot_name}_x" command_interface="cartesian_pose" index="0" />
     <xacro:general_purpose_io prefix="${robot_name}_y" command_interface="cartesian_pose" index="0" />
@@ -181,4 +221,5 @@
     <xacro:general_purpose_io prefix="${robot_name}_qy" command_interface="cartesian_pose" index="4" />
     <xacro:general_purpose_io prefix="${robot_name}_qz" command_interface="cartesian_pose" index="5" />
+    <!-- Cartesian velocity interfaces -->
     <xacro:general_purpose_io prefix="${robot_name}_vx" command_interface="cartesian_velocity"
       index="0" />
@@ -211,6 +252,6 @@
       </xacro:if>
     </hardware>
-    <xacro:interface_spawner robot_name="franka1" />
-    <xacro:interface_spawner robot_name="franka2" />
+    <xacro:interface_spawner robot_name="franka1" initial_j1="${pi/2}" />
+    <xacro:interface_spawner robot_name="franka2" initial_j1="${-pi/2}" />
   </ros2_control>
   <xacro:if value="$(arg gazebo)">
@@ -221,7 +262,4 @@
       </plugin>
     </gazebo>
-    <xacro:if value="$(arg hand)">
-      <!-- Symmetrical gripper is now handled by JointTrajectoryController in ros2_control -->
-    </xacro:if>
   </xacro:if>
 </robot>
