Commit message: Simulation Tests

File: src/franka_ros2_multimanual/idra_franka_launch/urdf/bimanual.urdf.xacro (robot description, xacro)
@@ -1,10 +1,10 @@
 <?xml version='1.0' encoding='utf-8'?>
 <robot xmlns:xacro="http://www.ros.org/wiki/xacro" name="idra_bimanual_setup">
-  <xacro:include filename="$(find franka_description)/robots/common/franka_robot.xacro"/>
-  <link name="world"/>
+  <xacro:include filename="$(find franka_description)/robots/common/franka_robot.xacro" />
+  <link name="world" />
   <joint name="world_joint" type="fixed">
-    <origin rpy="0 0 0" xyz="0 0 0.2"/>
-    <parent link="world"/>
-    <child link="table"/>
+    <origin rpy="0 0 0" xyz="0 0 0.2" />
+    <parent link="world" />
+    <child link="table" />
   </joint>
   <!--  _____     _     _       -->
@@ -15,22 +15,22 @@
   <!--                          -->
   <material name="tablematerial">
-    <color rgba="0.8 0.8 0.8 1.0"/>
+    <color rgba="0.8 0.8 0.8 1.0" />
   </material>
   <material name="platematerial">
-    <color rgba="0.85 0.85 0.85 1.0"/>
+    <color rgba="0.85 0.85 0.85 1.0" />
   </material>
   <link name="table">
     <visual>
       <geometry>
-        <box size="1.2 0.8 0.2"/>
-      </geometry>
-      <origin xyz="0.6 0.4 -0.1"/>
-      <material name="tablematerial"/>
+        <box size="1.2 0.8 0.2" />
+      </geometry>
+      <origin xyz="0.6 0.4 -0.1" />
+      <material name="tablematerial" />
     </visual>
     <collision>
       <geometry>
-        <box size="1.2 0.8 0.2"/>
-      </geometry>
-      <origin xyz="0.6 0.4 -0.1"/>
+        <box size="1.2 0.8 0.2" />
+      </geometry>
+      <origin xyz="0.6 0.4 -0.1" />
     </collision>
   </link>
@@ -38,28 +38,28 @@
     <visual>
       <geometry>
-        <box size="0.29 0.29 0.018"/>
-      </geometry>
-      <origin xyz="0.145 0.145 0.009"/>
-      <material name="platematerial"/>
+        <box size="0.29 0.29 0.018" />
+      </geometry>
+      <origin xyz="0.145 0.145 0.009" />
+      <material name="platematerial" />
     </visual>
   </link>
   <joint name="table_to_plate1" type="fixed">
-    <parent link="table"/>
-    <child link="robot1_plate"/>
-    <origin xyz="0.88 0.48 0.0"/>
+    <parent link="table" />
+    <child link="robot1_plate" />
+    <origin xyz="0.88 0.48 0.0" />
   </joint>
   <link name="robot2_plate">
     <visual>
       <geometry>
-        <box size="0.29 0.29 0.018"/>
-      </geometry>
-      <origin xyz="0.145 0.145 0.009"/>
-      <material name="platematerial"/>
+        <box size="0.29 0.29 0.018" />
+      </geometry>
+      <origin xyz="0.145 0.145 0.009" />
+      <material name="platematerial" />
     </visual>
   </link>
   <joint name="table_to_plate2" type="fixed">
-    <parent link="table"/>
-    <child link="robot2_plate"/>
-    <origin xyz="0.03 0.48 0.0"/>
+    <parent link="table" />
+    <child link="robot2_plate" />
+    <origin xyz="0.03 0.48 0.0" />
   </joint>
   <!--  _____                _           ____                                -->
@@ -90,5 +90,6 @@
   <xacro:arg name="franka1_ip" default="192.160.100.11" />
   <xacro:arg name="franka2_ip" default="192.160.100.12" />
-  <xacro:arg name="controller_path" default="$(find idra_franka_launch)/config/basic_controllers.yaml" />
+  <xacro:arg name="controller_path"
+    default="$(find idra_franka_launch)/config/basic_controllers.yaml" />
   <!--  _____                _         _  -->
   <!-- |  ___| __ __ _ _ __ | | ____ _/ | -->
@@ -98,29 +99,30 @@
   <!--                                    -->
   <xacro:franka_robot arm_id="fr3"
-                      joint_limits="${xacro.load_yaml('$(find franka_description)/robots/fr3/joint_limits.yaml')}"
-                      inertials="${xacro.load_yaml('$(find franka_description)/robots/fr3/inertials.yaml')}"
-                      kinematics="${xacro.load_yaml('$(find franka_description)/robots/fr3/kinematics.yaml')}"
-                      dynamics="${xacro.load_yaml('$(find franka_description)/robots/fr3/dynamics.yaml')}"
-                      gazebo="$(arg gazebo)"
-                      hand="$(arg hand)"
-                      ee_id="$(arg ee_id)"
-                      with_sc="$(arg with_sc)"
-                      ros2_control="$(arg ros2_control)"
-                      robot_ip="$(arg franka1_ip)"
-                      arm_prefix="franka1_"
-                      parent=""
-                      connected_to=""
-                      no_prefix="false"
-                      use_fake_hardware="$(arg use_fake_hardware)"
-                      fake_sensor_commands="$(arg fake_sensor_commands)"
-                      gazebo_effort="$(arg gazebo_effort)"
-                      rpy_ee="0 0 ${-pi/4}"
-                      >
+    joint_limits="${xacro.load_yaml('$(find franka_description)/robots/fr3/joint_limits.yaml')}"
+    inertials="${xacro.load_yaml('$(find franka_description)/robots/fr3/inertials.yaml')}"
+    kinematics="${xacro.load_yaml('$(find franka_description)/robots/fr3/kinematics.yaml')}"
+    dynamics="${xacro.load_yaml('$(find franka_description)/robots/fr3/dynamics.yaml')}"
+    gazebo="$(arg gazebo)"
+    hand="$(arg hand)"
+    ee_id="$(arg ee_id)"
+    with_sc="$(arg with_sc)"
+    ros2_control="$(arg ros2_control)"
+    robot_ip="$(arg franka1_ip)"
+    arm_prefix="franka1_"
+    parent=""
+    connected_to=""
+    no_prefix="false"
+    use_fake_hardware="$(arg use_fake_hardware)"
+    fake_sensor_commands="$(arg fake_sensor_commands)"
+    gazebo_effort="$(arg gazebo_effort)"
+    rpy_ee="0 0 ${-pi/4}"
+  >
   </xacro:franka_robot>
-  <!-- Dimensions taken from technical drawing of Franka plate and custom designed plate, do not touch -->
+  <!-- Dimensions taken from technical drawing of Franka plate and custom designed plate, do not
+  touch -->
   <joint name="plate_to_franka1" type="fixed">
-    <parent link="robot1_plate"/>
-    <child link="franka1_fr3_link0"/>
-    <origin xyz="0.145 0.107 0.018" rpy="0 0 ${-pi/2}"/>
+    <parent link="robot1_plate" />
+    <child link="franka1_fr3_link0" />
+    <origin xyz="0.145 0.107 0.018" rpy="0 0 ${-pi/2}" />
   </joint>
   <!--  _____                _         ____   -->
@@ -131,29 +133,30 @@
   <!--                                        -->
   <xacro:franka_robot arm_id="fr3"
-                      joint_limits="${xacro.load_yaml('$(find franka_description)/robots/fr3/joint_limits.yaml')}"
-                      inertials="${xacro.load_yaml('$(find franka_description)/robots/fr3/inertials.yaml')}"
-                      kinematics="${xacro.load_yaml('$(find franka_description)/robots/fr3/kinematics.yaml')}"
-                      dynamics="${xacro.load_yaml('$(find franka_description)/robots/fr3/dynamics.yaml')}"
-                      gazebo="$(arg gazebo)"
-                      hand="$(arg hand)"
-                      ee_id="$(arg ee_id)"
-                      with_sc="$(arg with_sc)"
-                      ros2_control="$(arg ros2_control)"
-                      robot_ip="$(arg franka2_ip)"
-                      arm_prefix="franka2_"
-                      parent=""
-                      connected_to=""
-                      no_prefix="false"
-                      use_fake_hardware="$(arg use_fake_hardware)"
-                      fake_sensor_commands="$(arg fake_sensor_commands)"
-                      gazebo_effort="$(arg gazebo_effort)"
-                      rpy_ee="0 0 ${-pi/4}"
-                      >
+    joint_limits="${xacro.load_yaml('$(find franka_description)/robots/fr3/joint_limits.yaml')}"
+    inertials="${xacro.load_yaml('$(find franka_description)/robots/fr3/inertials.yaml')}"
+    kinematics="${xacro.load_yaml('$(find franka_description)/robots/fr3/kinematics.yaml')}"
+    dynamics="${xacro.load_yaml('$(find franka_description)/robots/fr3/dynamics.yaml')}"
+    gazebo="$(arg gazebo)"
+    hand="$(arg hand)"
+    ee_id="$(arg ee_id)"
+    with_sc="$(arg with_sc)"
+    ros2_control="$(arg ros2_control)"
+    robot_ip="$(arg franka2_ip)"
+    arm_prefix="franka2_"
+    parent=""
+    connected_to=""
+    no_prefix="false"
+    use_fake_hardware="$(arg use_fake_hardware)"
+    fake_sensor_commands="$(arg fake_sensor_commands)"
+    gazebo_effort="$(arg gazebo_effort)"
+    rpy_ee="0 0 ${-pi/4}"
+  >
   </xacro:franka_robot>
-  <!-- Dimensions taken from technical drawing of Franka plate and custom designed plate, do not touch -->
+  <!-- Dimensions taken from technical drawing of Franka plate and custom designed plate, do not
+  touch -->
   <joint name="plate_to_franka2" type="fixed">
-    <parent link="robot2_plate"/>
-    <child link="franka2_fr3_link0"/>
-    <origin xyz="0.145 0.107 0.018" rpy="0 0 ${-pi/2}"/>
+    <parent link="robot2_plate" />
+    <child link="franka2_fr3_link0" />
+    <origin xyz="0.145 0.107 0.018" rpy="0 0 ${-pi/2}" />
   </joint>
   <!-- TODO: add if based on ros2_control arg -->
@@ -166,8 +169,8 @@
           https://github.com/ros-controls/gz_ros2_control/issues/343
           Command Interfaces -->
-          <command_interface name="position"/>
-          <command_interface name="velocity"/>
+        <command_interface name="position" />
+        <command_interface name="velocity" />
         <xacro:if value="$(eval not gazebo or gazebo_effort)">
-          <command_interface name="effort"/>
+          <command_interface name="effort" />
         </xacro:if>
         <!-- State Interfaces -->
@@ -175,51 +178,60 @@
           <param name="initial_value">${initial_position}</param>
         </state_interface>
-        <state_interface name="velocity"/>
-          <param name="initial_value">0.0</param>
-        <state_interface name="effort"/>
+        <state_interface name="velocity" />
+        <param name="initial_value">0.0</param>
+        <state_interface name="effort" />
       </joint>
     </xacro:macro>
     <xacro:macro name="general_purpose_io" params="prefix command_interface index">
       <gpio name="${prefix}">
-        <command_interface name="${command_interface}"/>
+        <command_interface name="${command_interface}" />
         <param name="index">${index}</param>
       </gpio>
     </xacro:macro>
-    <xacro:configure_joint joint_name="${robot_name}_fr3_joint1" initial_position="0.0"/>
-    <xacro:configure_joint joint_name="${robot_name}_fr3_joint2" initial_position="${-pi/4}"/>
-    <xacro:configure_joint joint_name="${robot_name}_fr3_joint3" initial_position="0.0"/>
-    <xacro:configure_joint joint_name="${robot_name}_fr3_joint4" initial_position="${-3*pi/4}"/>
-    <xacro:configure_joint joint_name="${robot_name}_fr3_joint5" initial_position="0.0"/>
-    <xacro:configure_joint joint_name="${robot_name}_fr3_joint6" initial_position="${pi/2}"/>
-    <xacro:configure_joint joint_name="${robot_name}_fr3_joint7" initial_position="${pi/4}"/>
+    <xacro:configure_joint joint_name="${robot_name}_fr3_joint1" initial_position="0.0" />
+    <xacro:configure_joint joint_name="${robot_name}_fr3_joint2" initial_position="${-pi/4}" />
+    <xacro:configure_joint joint_name="${robot_name}_fr3_joint3" initial_position="0.0" />
+    <xacro:configure_joint joint_name="${robot_name}_fr3_joint4" initial_position="${-3*pi/4}" />
+    <xacro:configure_joint joint_name="${robot_name}_fr3_joint5" initial_position="0.0" />
+    <xacro:configure_joint joint_name="${robot_name}_fr3_joint6" initial_position="${pi/2}" />
+    <xacro:configure_joint joint_name="${robot_name}_fr3_joint7" initial_position="${pi/4}" />
     <xacro:if value="$(eval gazebo and hand)">
       <xacro:configure_joint joint_name="${robot_name}_fr3_finger_joint1" initial_position="0.0" />
     </xacro:if>
     <!-- Elbow interfaces -->
-    <xacro:general_purpose_io prefix="${robot_name}_joint_3_position" command_interface="elbow_command" index="0"/>
-    <xacro:general_purpose_io prefix="${robot_name}_joint_4_sign" command_interface="elbow_command" index="1"/>
+    <xacro:general_purpose_io prefix="${robot_name}_joint_3_position"
+      command_interface="elbow_command" index="0" />
+    <xacro:general_purpose_io prefix="${robot_name}_joint_4_sign" command_interface="elbow_command"
+      index="1" />
     <!-- Cartesian position interfaces -->
     <xacro:macro name="loop" params="i">
       <xacro:unless value="${i == 16}">
-        <xacro:general_purpose_io prefix="${robot_name}_${i}" command_interface="cartesian_pose_command" index="${i}"/>
-        <xacro:loop i="${i+1}"/>
+        <xacro:general_purpose_io prefix="${robot_name}_${i}"
+          command_interface="cartesian_pose_command" index="${i}" />
+        <xacro:loop i="${i+1}" />
       </xacro:unless>
     </xacro:macro>
-    <xacro:loop i="0"/>
+    <xacro:loop i="0" />
     <!-- Cartesian pose (position + quaternion) interface -->
-    <xacro:general_purpose_io prefix="${robot_name}_x"  command_interface="cartesian_pose" index="0"/>
-    <xacro:general_purpose_io prefix="${robot_name}_y"  command_interface="cartesian_pose" index="0"/>
-    <xacro:general_purpose_io prefix="${robot_name}_z"  command_interface="cartesian_pose" index="1"/>
-    <xacro:general_purpose_io prefix="${robot_name}_qw" command_interface="cartesian_pose" index="2"/>
-    <xacro:general_purpose_io prefix="${robot_name}_qx" command_interface="cartesian_pose" index="3"/>
-    <xacro:general_purpose_io prefix="${robot_name}_qy" command_interface="cartesian_pose" index="4"/>
-    <xacro:general_purpose_io prefix="${robot_name}_qz" command_interface="cartesian_pose" index="5"/>
+    <xacro:general_purpose_io prefix="${robot_name}_x" command_interface="cartesian_pose" index="0" />
+    <xacro:general_purpose_io prefix="${robot_name}_y" command_interface="cartesian_pose" index="0" />
+    <xacro:general_purpose_io prefix="${robot_name}_z" command_interface="cartesian_pose" index="1" />
+    <xacro:general_purpose_io prefix="${robot_name}_qw" command_interface="cartesian_pose" index="2" />
+    <xacro:general_purpose_io prefix="${robot_name}_qx" command_interface="cartesian_pose" index="3" />
+    <xacro:general_purpose_io prefix="${robot_name}_qy" command_interface="cartesian_pose" index="4" />
+    <xacro:general_purpose_io prefix="${robot_name}_qz" command_interface="cartesian_pose" index="5" />
     <!-- Cartesian velocity interfaces -->
-    <xacro:general_purpose_io prefix="${robot_name}_vx" command_interface="cartesian_velocity" index="0"/>
-    <xacro:general_purpose_io prefix="${robot_name}_vy" command_interface="cartesian_velocity" index="1"/>
-    <xacro:general_purpose_io prefix="${robot_name}_vz" command_interface="cartesian_velocity" index="2"/>
-    <xacro:general_purpose_io prefix="${robot_name}_wx" command_interface="cartesian_velocity" index="3"/>
-    <xacro:general_purpose_io prefix="${robot_name}_wy" command_interface="cartesian_velocity" index="4"/>
-    <xacro:general_purpose_io prefix="${robot_name}_wz" command_interface="cartesian_velocity" index="5"/>
+    <xacro:general_purpose_io prefix="${robot_name}_vx" command_interface="cartesian_velocity"
+      index="0" />
+    <xacro:general_purpose_io prefix="${robot_name}_vy" command_interface="cartesian_velocity"
+      index="1" />
+    <xacro:general_purpose_io prefix="${robot_name}_vz" command_interface="cartesian_velocity"
+      index="2" />
+    <xacro:general_purpose_io prefix="${robot_name}_wx" command_interface="cartesian_velocity"
+      index="3" />
+    <xacro:general_purpose_io prefix="${robot_name}_wy" command_interface="cartesian_velocity"
+      index="4" />
+    <xacro:general_purpose_io prefix="${robot_name}_wz" command_interface="cartesian_velocity"
+      index="5" />
   </xacro:macro>
   <ros2_control name="FrankaMultimanualHardwareInterface" type="system">
@@ -240,13 +252,14 @@
       </xacro:if>
     </hardware>
-    <xacro:interface_spawner robot_name="franka1"/>
-    <xacro:interface_spawner robot_name="franka2"/>
+    <xacro:interface_spawner robot_name="franka1" />
+    <xacro:interface_spawner robot_name="franka2" />
   </ros2_control>
   <xacro:if value="$(arg gazebo)">
-  <gazebo>
-    <plugin filename="franka_ign_ros2_control-system" name="ign_ros2_control::IgnitionROS2ControlPlugin">
-      <parameters>$(arg controller_path)</parameters>
-    </plugin>
-  </gazebo>
+    <gazebo>
+      <plugin filename="franka_ign_ros2_control-system"
+        name="ign_ros2_control::IgnitionROS2ControlPlugin">
+        <parameters>$(arg controller_path)</parameters>
+      </plugin>
+    </gazebo>
   </xacro:if>
 </robot>

Commit message: still unconsistent

File: src/franka_manipulation_env/urdf/bimanual_custom.urdf.xacro (robot description, xacro)
@@ -17,14 +17,14 @@
     <visual>
       <geometry>
-        <box size="1.2 0.8 0.2" />
-      </geometry>
-      <origin xyz="0.6 0.4 -0.1" />
+        <box size="0.8 1.6 0.04" />
+      </geometry>
+      <origin xyz="0 0 -0.02" />
       <material name="tablematerial" />
     </visual>
     <collision>
       <geometry>
-        <box size="1.2 0.8 0.2" />
-      </geometry>
-      <origin xyz="0.6 0.4 -0.1" />
+        <box size="0.8 1.6 0.04" />
+      </geometry>
+      <origin xyz="0 0 -0.02" />
     </collision>
   </link>
@@ -41,5 +41,5 @@
     <parent link="table" />
     <child link="robot1_plate" />
-    <origin xyz="0.88 0.48 0.0" />
+    <origin xyz="-0.2 0.6 0.0" />
   </joint>
   <link name="robot2_plate">
@@ -55,5 +55,5 @@
     <parent link="table" />
     <child link="robot2_plate" />
-    <origin xyz="0.03 0.48 0.0" />
+    <origin xyz="-0.2 -0.6 0.0" />
   </joint>
   <!-- Configuration Arguments -->
@@ -123,5 +123,5 @@
     <parent link="robot2_plate" />
     <child link="franka2_fr3_link0" />
-    <origin xyz="0.145 0.107 0.018" rpy="0 0 ${-pi/2}" />
+    <origin xyz="0.145 0.107 0.018" rpy="0 0 ${pi/2}" />
   </joint>
   <!-- Hardware Interface Spawner -->

Commit message: Parallel execution

File: src/franka_manipulation_env/urdf/bimanual_custom.urdf.xacro (robot description, xacro)
@@ -62,4 +62,23 @@
     <child link="robot2_plate" />
     <origin xyz="0.03 0.48 0.0" />
+  </joint>
+  <!-- SEMANTIC TARGET FRAMES (For MoveIt & Orchestrator) -->
+  <link name="shared" />
+  <joint name="table_to_shared" type="fixed">
+    <parent link="table" />
+    <child link="shared" />
+    <origin xyz="0.45 0.4 0.025" rpy="0 0 0" />
+  </joint>
+  <link name="box" />
+  <joint name="table_to_box" type="fixed">
+    <parent link="table" />
+    <child link="box" />
+    <origin xyz="0.1 0.1 0.03" rpy="0 0 0" />
+  </joint>
+  <link name="base_pose" />
+  <joint name="table_to_base" type="fixed">
+    <parent link="table" />
+    <child link="base_pose" />
+    <origin xyz="1.1 0.2 0.025" rpy="0 0 0" />
   </joint>
   <!--  _____                _           ____                                -->
@@ -253,6 +272,6 @@
       </xacro:if>
     </hardware>
-    <xacro:interface_spawner robot_name="franka1" initial_j1="${pi/2}" />
-    <xacro:interface_spawner robot_name="franka2" initial_j1="${-pi/2}" />
+    <xacro:interface_spawner robot_name="franka1" initial_j1="0.0" />
+    <xacro:interface_spawner robot_name="franka2" initial_j1="0.0" />
   </ros2_control>
   <xacro:if value="$(arg gazebo)">
@@ -264,3 +283,18 @@
     </gazebo>
   </xacro:if>
+  <!-- Gazebo Friction & Physics Overrides for Fingers -->
+  <xacro:macro name="finger_gazebo" params="arm_id finger_id">
+    <gazebo reference="${arm_id}_fr3_finger_joint${finger_id}">
+      <mu1>1000.0</mu1>
+      <mu2>1000.0</mu2>
+      <kp>1000000.0</kp>
+      <kd>1.0</kd>
+      <minDepth>0.001</minDepth>
+      <maxVel>0.1</maxVel>
+    </gazebo>
+  </xacro:macro>
+  <xacro:finger_gazebo arm_id="franka1" finger_id="1" />
+  <xacro:finger_gazebo arm_id="franka1" finger_id="2" />
+  <xacro:finger_gazebo arm_id="franka2" finger_id="1" />
+  <xacro:finger_gazebo arm_id="franka2" finger_id="2" />
 </robot>

Commit message: sim allineata

File: src/franka_manipulation_env/urdf/bimanual_custom.urdf.xacro (robot description, xacro)
@@ -43,4 +43,10 @@
       <material name="platematerial" />
     </visual>
+    <collision>
+      <geometry>
+        <box size="0.29 0.29 0.018" />
+      </geometry>
+      <origin xyz="0.145 0.145 0.009" />
+    </collision>
   </link>
   <joint name="table_to_plate1" type="fixed">
@@ -57,4 +63,10 @@
       <material name="platematerial" />
     </visual>
+    <collision>
+      <geometry>
+        <box size="0.29 0.29 0.018" />
+      </geometry>
+      <origin xyz="0.145 0.145 0.009" />
+    </collision>
   </link>
   <joint name="table_to_plate2" type="fixed">

File: src/franka_ros2_multimanual/idra_franka_launch/urdf/bimanual.urdf.xacro (robot description, xacro)
@@ -43,4 +43,10 @@
       <material name="platematerial" />
     </visual>
+    <collision>
+      <geometry>
+        <box size="0.29 0.29 0.018" />
+      </geometry>
+      <origin xyz="0.145 0.145 0.009" />
+    </collision>
   </link>
   <joint name="table_to_plate1" type="fixed">
@@ -57,4 +63,10 @@
       <material name="platematerial" />
     </visual>
+    <collision>
+      <geometry>
+        <box size="0.29 0.29 0.018" />
+      </geometry>
+      <origin xyz="0.145 0.145 0.009" />
+    </collision>
   </link>
   <joint name="table_to_plate2" type="fixed">
