Commit message: BT PER REA

File: src/franka_manipulation_env/srdf/bimanual_sim_srdf.xacro (robot description, xacro)
@@ -7,133 +7,152 @@
   </group>
   <group name="franka1_arm">
-    <chain base_link="franka1_fr3_link0" tip_link="franka1_fr3_link8"/>
+    <chain base_link="franka1_fr3_link0" tip_link="franka1_fr3_link8" />
   </group>
   <group name="franka1_hand">
-    <link name="franka1_fr3_hand"/>
-    <link name="franka1_fr3_leftfinger"/>
-    <link name="franka1_fr3_rightfinger"/>
-    <joint name="franka1_fr3_finger_joint1"/>
-    <joint name="franka1_fr3_finger_joint2"/>
+    <link name="franka1_fr3_hand" />
+    <link name="franka1_fr3_leftfinger" />
+    <link name="franka1_fr3_rightfinger" />
+    <joint name="franka1_fr3_finger_joint1" />
+    <joint name="franka1_fr3_finger_joint2" />
   </group>
   <group name="franka1_manipulator">
-    <chain base_link="franka1_fr3_link0" tip_link="franka1_fr3_hand_tcp"/>
+    <chain base_link="franka1_fr3_link0" tip_link="franka1_fr3_hand_tcp" />
   </group>
   <group_state name="open" group="franka1_hand">
-    <joint name="franka1_fr3_finger_joint1" value="0.035"/>
-    <joint name="franka1_fr3_finger_joint2" value="0.035"/>
+    <joint name="franka1_fr3_finger_joint1" value="0.035" />
+    <joint name="franka1_fr3_finger_joint2" value="0.035" />
   </group_state>
   <group_state name="close" group="franka1_hand">
-    <joint name="franka1_fr3_finger_joint1" value="0"/>
-    <joint name="franka1_fr3_finger_joint2" value="0"/>
+    <joint name="franka1_fr3_finger_joint1" value="0" />
+    <joint name="franka1_fr3_finger_joint2" value="0" />
   </group_state>
-  <end_effector name="franka1_hand_tcp" parent_link="franka1_fr3_hand_tcp" group="franka1_hand" parent_group="franka1_manipulator"/>
-  <end_effector name="franka1_hand" parent_link="franka1_fr3_link8" group="franka1_hand" parent_group="franka1_arm"/>
+  <end_effector name="franka1_hand_tcp" parent_link="franka1_fr3_hand_tcp" group="franka1_hand"
+    parent_group="franka1_manipulator" />
+  <end_effector name="franka1_hand" parent_link="franka1_fr3_link8" group="franka1_hand"
+    parent_group="franka1_arm" />
   <group name="franka2_arm">
-    <chain base_link="franka2_fr3_link0" tip_link="franka2_fr3_link8"/>
+    <chain base_link="franka2_fr3_link0" tip_link="franka2_fr3_link8" />
   </group>
   <group name="franka2_hand">
-    <link name="franka2_fr3_hand"/>
-    <link name="franka2_fr3_leftfinger"/>
-    <link name="franka2_fr3_rightfinger"/>
-    <joint name="franka2_fr3_finger_joint1"/>
-    <joint name="franka2_fr3_finger_joint2"/>
+    <link name="franka2_fr3_hand" />
+    <link name="franka2_fr3_leftfinger" />
+    <link name="franka2_fr3_rightfinger" />
+    <joint name="franka2_fr3_finger_joint1" />
+    <joint name="franka2_fr3_finger_joint2" />
   </group>
   <group name="franka2_manipulator">
-    <chain base_link="franka2_fr3_link0" tip_link="franka2_fr3_hand_tcp"/>
+    <chain base_link="franka2_fr3_link0" tip_link="franka2_fr3_hand_tcp" />
   </group>
+  <group name="bimanual_manipulator">
+    <chain base_link="franka1_fr3_link0" tip_link="franka1_fr3_hand_tcp" />
+    <chain base_link="franka2_fr3_link0" tip_link="franka2_fr3_hand_tcp" />
+  </group>
+  <end_effector name="bimanual_grasp"
+    parent_link="franka1_fr3_hand_tcp"
+    group="bimanual" />
   <group_state name="open" group="franka2_hand">
-    <joint name="franka2_fr3_finger_joint1" value="0.035"/>
-    <joint name="franka2_fr3_finger_joint2" value="0.035"/>
+    <joint name="franka2_fr3_finger_joint1" value="0.035" />
+    <joint name="franka2_fr3_finger_joint2" value="0.035" />
   </group_state>
   <group_state name="close" group="franka2_hand">
-    <joint name="franka2_fr3_finger_joint1" value="0"/>
-    <joint name="franka2_fr3_finger_joint2" value="0"/>
+    <joint name="franka2_fr3_finger_joint1" value="0" />
+    <joint name="franka2_fr3_finger_joint2" value="0" />
   </group_state>
-  <end_effector name="franka2_hand_tcp" parent_link="franka2_fr3_hand_tcp" group="franka2_hand" parent_group="franka2_manipulator"/>
-  <end_effector name="franka2_hand" parent_link="franka2_fr3_link8" group="franka2_hand" parent_group="franka2_arm"/>
-  <disable_collisions link1="franka1_fr3_link0" link2="franka1_fr3_link1" reason="Adjacent"/>
-  <disable_collisions link1="franka1_fr3_link0" link2="franka1_fr3_link2" reason="Never"/>
-  <disable_collisions link1="franka1_fr3_link0" link2="franka1_fr3_link3" reason="Never"/>
-  <disable_collisions link1="franka1_fr3_link0" link2="franka1_fr3_link4" reason="Never"/>
-  <disable_collisions link1="franka1_fr3_link1" link2="franka1_fr3_link2" reason="Adjacent"/>
-  <disable_collisions link1="franka1_fr3_link1" link2="franka1_fr3_link3" reason="Never"/>
-  <disable_collisions link1="franka1_fr3_link1" link2="franka1_fr3_link4" reason="Never"/>
-  <disable_collisions link1="franka1_fr3_link2" link2="franka1_fr3_link3" reason="Adjacent"/>
-  <disable_collisions link1="franka1_fr3_link2" link2="franka1_fr3_link4" reason="Never"/>
-  <disable_collisions link1="franka1_fr3_link2" link2="franka1_fr3_link6" reason="Never"/>
-  <disable_collisions link1="franka1_fr3_link3" link2="franka1_fr3_link4" reason="Adjacent"/>
-  <disable_collisions link1="franka1_fr3_link3" link2="franka1_fr3_link5" reason="Never"/>
-  <disable_collisions link1="franka1_fr3_link3" link2="franka1_fr3_link6" reason="Never"/>
-  <disable_collisions link1="franka1_fr3_link3" link2="franka1_fr3_link7" reason="Never"/>
-  <disable_collisions link1="franka1_fr3_link4" link2="franka1_fr3_link5" reason="Adjacent"/>
-  <disable_collisions link1="franka1_fr3_link4" link2="franka1_fr3_link6" reason="Never"/>
-  <disable_collisions link1="franka1_fr3_link4" link2="franka1_fr3_link7" reason="Never"/>
-  <disable_collisions link1="franka1_fr3_link4" link2="franka1_fr3_link8" reason="Never"/>
-  <disable_collisions link1="franka1_fr3_link5" link2="franka1_fr3_link6" reason="Adjacent"/>
-  <disable_collisions link1="franka1_fr3_link6" link2="franka1_fr3_link7" reason="Adjacent"/>
-  <disable_collisions link1="franka1_fr3_link6" link2="franka1_fr3_link8" reason="Default"/>
-  <disable_collisions link1="franka1_fr3_link7" link2="franka1_fr3_link8" reason="Adjacent"/>
-  <disable_collisions link1="franka1_fr3_hand" link2="franka1_fr3_link3" reason="Never"/>
-  <disable_collisions link1="franka1_fr3_hand" link2="franka1_fr3_link4" reason="Never"/>
-  <disable_collisions link1="franka1_fr3_hand" link2="franka1_fr3_link6" reason="Never"/>
-  <disable_collisions link1="franka1_fr3_hand" link2="franka1_fr3_link7" reason="Adjacent"/>
-  <disable_collisions link1="franka1_fr3_hand" link2="franka1_fr3_link8" reason="Adjacent"/>
-  <disable_collisions link1="franka1_fr3_leftfinger" link2="franka1_fr3_link3" reason="Never"/>
-  <disable_collisions link1="franka1_fr3_leftfinger" link2="franka1_fr3_link4" reason="Never"/>
-  <disable_collisions link1="franka1_fr3_leftfinger" link2="franka1_fr3_link6" reason="Never"/>
-  <disable_collisions link1="franka1_fr3_leftfinger" link2="franka1_fr3_link7" reason="Never"/>
-  <disable_collisions link1="franka1_fr3_leftfinger" link2="franka1_fr3_link8" reason="Never"/>
-  <disable_collisions link1="franka1_fr3_link3" link2="franka1_fr3_rightfinger" reason="Never"/>
-  <disable_collisions link1="franka1_fr3_link4" link2="franka1_fr3_rightfinger" reason="Never"/>
-  <disable_collisions link1="franka1_fr3_link6" link2="franka1_fr3_rightfinger" reason="Never"/>
-  <disable_collisions link1="franka1_fr3_link7" link2="franka1_fr3_rightfinger" reason="Never"/>
-  <disable_collisions link1="franka1_fr3_link8" link2="franka1_fr3_rightfinger" reason="Never"/>
-  <disable_collisions link1="franka1_fr3_hand" link2="franka1_plate" reason="Never" />
-  <disable_collisions link1="franka2_fr3_link0" link2="franka2_fr3_link1" reason="Adjacent"/>
-  <disable_collisions link1="franka2_fr3_link0" link2="franka2_fr3_link2" reason="Never"/>
-  <disable_collisions link1="franka2_fr3_link0" link2="franka2_fr3_link3" reason="Never"/>
-  <disable_collisions link1="franka2_fr3_link0" link2="franka2_fr3_link4" reason="Never"/>
-  <disable_collisions link1="franka2_fr3_link1" link2="franka2_fr3_link2" reason="Adjacent"/>
-  <disable_collisions link1="franka2_fr3_link1" link2="franka2_fr3_link3" reason="Never"/>
-  <disable_collisions link1="franka2_fr3_link1" link2="franka2_fr3_link4" reason="Never"/>
-  <disable_collisions link1="franka2_fr3_link2" link2="franka2_fr3_link3" reason="Adjacent"/>
-  <disable_collisions link1="franka2_fr3_link2" link2="franka2_fr3_link4" reason="Never"/>
-  <disable_collisions link1="franka2_fr3_link2" link2="franka2_fr3_link6" reason="Never"/>
-  <disable_collisions link1="franka2_fr3_link3" link2="franka2_fr3_link4" reason="Adjacent"/>
-  <disable_collisions link1="franka2_fr3_link3" link2="franka2_fr3_link5" reason="Never"/>
-  <disable_collisions link1="franka2_fr3_link3" link2="franka2_fr3_link6" reason="Never"/>
-  <disable_collisions link1="franka2_fr3_link3" link2="franka2_fr3_link7" reason="Never"/>
-  <disable_collisions link1="franka2_fr3_link4" link2="franka2_fr3_link5" reason="Adjacent"/>
-  <disable_collisions link1="franka2_fr3_link4" link2="franka2_fr3_link6" reason="Never"/>
-  <disable_collisions link1="franka2_fr3_link4" link2="franka2_fr3_link7" reason="Never"/>
-  <disable_collisions link1="franka2_fr3_link4" link2="franka2_fr3_link8" reason="Never"/>
-  <disable_collisions link1="franka2_fr3_link5" link2="franka2_fr3_link6" reason="Adjacent"/>
-  <disable_collisions link1="franka2_fr3_link6" link2="franka2_fr3_link7" reason="Adjacent"/>
-  <disable_collisions link1="franka2_fr3_link6" link2="franka2_fr3_link8" reason="Default"/>
-  <disable_collisions link1="franka2_fr3_link7" link2="franka2_fr3_link8" reason="Adjacent"/>
-  <disable_collisions link1="franka2_fr3_hand" link2="franka2_fr3_link3" reason="Never"/>
-  <disable_collisions link1="franka2_fr3_hand" link2="franka2_fr3_link4" reason="Never"/>
-  <disable_collisions link1="franka2_fr3_hand" link2="franka2_fr3_link6" reason="Never"/>
-  <disable_collisions link1="franka2_fr3_hand" link2="franka2_fr3_link7" reason="Adjacent"/>
-  <disable_collisions link1="franka2_fr3_hand" link2="franka2_fr3_link8" reason="Adjacent"/>
-  <disable_collisions link1="franka2_fr3_leftfinger" link2="franka2_fr3_link3" reason="Never"/>
-  <disable_collisions link1="franka2_fr3_leftfinger" link2="franka2_fr3_link4" reason="Never"/>
-  <disable_collisions link1="franka2_fr3_leftfinger" link2="franka2_fr3_link6" reason="Never"/>
-  <disable_collisions link1="franka2_fr3_leftfinger" link2="franka2_fr3_link7" reason="Never"/>
-  <disable_collisions link1="franka2_fr3_leftfinger" link2="franka2_fr3_link8" reason="Never"/>
-  <disable_collisions link1="franka2_fr3_link3" link2="franka2_fr3_rightfinger" reason="Never"/>
-  <disable_collisions link1="franka2_fr3_link4" link2="franka2_fr3_rightfinger" reason="Never"/>
-  <disable_collisions link1="franka2_fr3_link6" link2="franka2_fr3_rightfinger" reason="Never"/>
-  <disable_collisions link1="franka2_fr3_link7" link2="franka2_fr3_rightfinger" reason="Never"/>
-  <disable_collisions link1="franka2_fr3_link8" link2="franka2_fr3_rightfinger" reason="Never"/>
-  <disable_collisions link1="franka2_fr3_hand" link2="franka2_plate" reason="Never" />
-  <disable_collisions link1="table" link2="robot1_plate" reason="Adjacent"/>
-  <disable_collisions link1="table" link2="robot2_plate" reason="Adjacent"/>
-  <disable_collisions link1="franka1_fr3_link0" link2="robot1_plate" reason="Adjacent"/>
-  <disable_collisions link1="franka2_fr3_link0" link2="robot2_plate" reason="Adjacent"/>
-  <disable_collisions link1="franka1_fr3_link0" link2="table" reason="Never"/>
-  <disable_collisions link1="franka2_fr3_link0" link2="table" reason="Never"/>
-  <disable_collisions link1="franka1_fr3_link1" link2="table" reason="Never"/>
-  <disable_collisions link1="franka2_fr3_link1" link2="table" reason="Never"/>
-  <disable_collisions link1="franka1_fr3_link0" link2="franka2_fr3_link0" reason="Adjacent"/>
+  <end_effector name="franka2_hand_tcp" parent_link="franka2_fr3_hand_tcp" group="franka2_hand"
+    parent_group="franka2_manipulator" />
+  <end_effector name="franka2_hand" parent_link="franka2_fr3_link8" group="franka2_hand"
+    parent_group="franka2_arm" />
+  <disable_collisions link1="franka1_fr3_link0" link2="franka1_fr3_link1" reason="Adjacent" />
+  <disable_collisions link1="franka1_fr3_link0" link2="franka1_fr3_link2" reason="Never" />
+  <disable_collisions link1="franka1_fr3_link0" link2="franka1_fr3_link3" reason="Never" />
+  <disable_collisions link1="franka1_fr3_link0" link2="franka1_fr3_link4" reason="Never" />
+  <disable_collisions link1="franka1_fr3_link1" link2="franka1_fr3_link2" reason="Adjacent" />
+  <disable_collisions link1="franka1_fr3_link1" link2="franka1_fr3_link3" reason="Never" />
+  <disable_collisions link1="franka1_fr3_link1" link2="franka1_fr3_link4" reason="Never" />
+  <disable_collisions link1="franka1_fr3_link2" link2="franka1_fr3_link3" reason="Adjacent" />
+  <disable_collisions link1="franka1_fr3_link2" link2="franka1_fr3_link4" reason="Never" />
+  <disable_collisions link1="franka1_fr3_link2" link2="franka1_fr3_link6" reason="Never" />
+  <disable_collisions link1="franka1_fr3_link3" link2="franka1_fr3_link4" reason="Adjacent" />
+  <disable_collisions link1="franka1_fr3_link3" link2="franka1_fr3_link5" reason="Never" />
+  <disable_collisions link1="franka1_fr3_link3" link2="franka1_fr3_link6" reason="Never" />
+  <disable_collisions link1="franka1_fr3_link3" link2="franka1_fr3_link7" reason="Never" />
+  <disable_collisions link1="franka1_fr3_link4" link2="franka1_fr3_link5" reason="Adjacent" />
+  <disable_collisions link1="franka1_fr3_link4" link2="franka1_fr3_link6" reason="Never" />
+  <disable_collisions link1="franka1_fr3_link4" link2="franka1_fr3_link7" reason="Never" />
+  <disable_collisions link1="franka1_fr3_link4" link2="franka1_fr3_link8" reason="Never" />
+  <disable_collisions link1="franka1_fr3_link5" link2="franka1_fr3_link6" reason="Adjacent" />
+  <disable_collisions link1="franka1_fr3_link6" link2="franka1_fr3_link7" reason="Adjacent" />
+  <disable_collisions link1="franka1_fr3_link6" link2="franka1_fr3_link8" reason="Default" />
+  <disable_collisions link1="franka1_fr3_link7" link2="franka1_fr3_link8" reason="Adjacent" />
+  <disable_collisions link1="franka1_fr3_hand" link2="franka1_fr3_link3" reason="Never" />
+  <disable_collisions link1="franka1_fr3_hand" link2="franka1_fr3_link4" reason="Never" />
+  <disable_collisions link1="franka1_fr3_hand" link2="franka1_fr3_link6" reason="Never" />
+  <disable_collisions link1="franka1_fr3_hand" link2="franka1_fr3_link7" reason="Adjacent" />
+  <disable_collisions link1="franka1_fr3_hand" link2="franka1_fr3_link8" reason="Adjacent" />
+  <disable_collisions link1="franka1_fr3_leftfinger" link2="franka1_fr3_link3" reason="Never" />
+  <disable_collisions link1="franka1_fr3_leftfinger" link2="franka1_fr3_link4" reason="Never" />
+  <disable_collisions link1="franka1_fr3_leftfinger" link2="franka1_fr3_link6" reason="Never" />
+  <disable_collisions link1="franka1_fr3_leftfinger" link2="franka1_fr3_link7" reason="Never" />
+  <disable_collisions link1="franka1_fr3_leftfinger" link2="franka1_fr3_link8" reason="Never" />
+  <disable_collisions link1="franka1_fr3_link3" link2="franka1_fr3_rightfinger" reason="Never" />
+  <disable_collisions link1="franka1_fr3_link4" link2="franka1_fr3_rightfinger" reason="Never" />
+  <disable_collisions link1="franka1_fr3_link6" link2="franka1_fr3_rightfinger" reason="Never" />
+  <disable_collisions link1="franka1_fr3_link7" link2="franka1_fr3_rightfinger" reason="Never" />
+  <disable_collisions link1="franka1_fr3_link8" link2="franka1_fr3_rightfinger" reason="Never" />
+  <disable_collisions link1="franka1_fr3_hand" link2="robot1_plate" reason="Never" />
+  <disable_collisions link1="franka1_fr3_leftfinger" link2="franka1_fr3_rightfinger"
+    reason="Default" />
+  <disable_collisions link1="franka1_fr3_hand" link2="franka1_fr3_leftfinger" reason="Adjacent" />
+  <disable_collisions link1="franka1_fr3_hand" link2="franka1_fr3_rightfinger" reason="Adjacent" />
+  <disable_collisions link1="franka2_fr3_link0" link2="franka2_fr3_link1" reason="Adjacent" />
+  <disable_collisions link1="franka2_fr3_link0" link2="franka2_fr3_link2" reason="Never" />
+  <disable_collisions link1="franka2_fr3_link0" link2="franka2_fr3_link3" reason="Never" />
+  <disable_collisions link1="franka2_fr3_link0" link2="franka2_fr3_link4" reason="Never" />
+  <disable_collisions link1="franka2_fr3_link1" link2="franka2_fr3_link2" reason="Adjacent" />
+  <disable_collisions link1="franka2_fr3_link1" link2="franka2_fr3_link3" reason="Never" />
+  <disable_collisions link1="franka2_fr3_link1" link2="franka2_fr3_link4" reason="Never" />
+  <disable_collisions link1="franka2_fr3_link2" link2="franka2_fr3_link3" reason="Adjacent" />
+  <disable_collisions link1="franka2_fr3_link2" link2="franka2_fr3_link4" reason="Never" />
+  <disable_collisions link1="franka2_fr3_link2" link2="franka2_fr3_link6" reason="Never" />
+  <disable_collisions link1="franka2_fr3_link3" link2="franka2_fr3_link4" reason="Adjacent" />
+  <disable_collisions link1="franka2_fr3_link3" link2="franka2_fr3_link5" reason="Never" />
+  <disable_collisions link1="franka2_fr3_link3" link2="franka2_fr3_link6" reason="Never" />
+  <disable_collisions link1="franka2_fr3_link3" link2="franka2_fr3_link7" reason="Never" />
+  <disable_collisions link1="franka2_fr3_link4" link2="franka2_fr3_link5" reason="Adjacent" />
+  <disable_collisions link1="franka2_fr3_link4" link2="franka2_fr3_link6" reason="Never" />
+  <disable_collisions link1="franka2_fr3_link4" link2="franka2_fr3_link7" reason="Never" />
+  <disable_collisions link1="franka2_fr3_link4" link2="franka2_fr3_link8" reason="Never" />
+  <disable_collisions link1="franka2_fr3_link5" link2="franka2_fr3_link6" reason="Adjacent" />
+  <disable_collisions link1="franka2_fr3_link6" link2="franka2_fr3_link7" reason="Adjacent" />
+  <disable_collisions link1="franka2_fr3_link6" link2="franka2_fr3_link8" reason="Default" />
+  <disable_collisions link1="franka2_fr3_link7" link2="franka2_fr3_link8" reason="Adjacent" />
+  <disable_collisions link1="franka2_fr3_hand" link2="franka2_fr3_link3" reason="Never" />
+  <disable_collisions link1="franka2_fr3_hand" link2="franka2_fr3_link4" reason="Never" />
+  <disable_collisions link1="franka2_fr3_hand" link2="franka2_fr3_link6" reason="Never" />
+  <disable_collisions link1="franka2_fr3_hand" link2="franka2_fr3_link7" reason="Adjacent" />
+  <disable_collisions link1="franka2_fr3_hand" link2="franka2_fr3_link8" reason="Adjacent" />
+  <disable_collisions link1="franka2_fr3_leftfinger" link2="franka2_fr3_link3" reason="Never" />
+  <disable_collisions link1="franka2_fr3_leftfinger" link2="franka2_fr3_link4" reason="Never" />
+  <disable_collisions link1="franka2_fr3_leftfinger" link2="franka2_fr3_link6" reason="Never" />
+  <disable_collisions link1="franka2_fr3_leftfinger" link2="franka2_fr3_link7" reason="Never" />
+  <disable_collisions link1="franka2_fr3_leftfinger" link2="franka2_fr3_link8" reason="Never" />
+  <disable_collisions link1="franka2_fr3_link3" link2="franka2_fr3_rightfinger" reason="Never" />
+  <disable_collisions link1="franka2_fr3_link4" link2="franka2_fr3_rightfinger" reason="Never" />
+  <disable_collisions link1="franka2_fr3_link6" link2="franka2_fr3_rightfinger" reason="Never" />
+  <disable_collisions link1="franka2_fr3_link7" link2="franka2_fr3_rightfinger" reason="Never" />
+  <disable_collisions link1="franka2_fr3_link8" link2="franka2_fr3_rightfinger" reason="Never" />
+  <disable_collisions link1="franka2_fr3_hand" link2="robot2_plate" reason="Never" />
+  <disable_collisions link1="franka2_fr3_leftfinger" link2="franka2_fr3_rightfinger"
+    reason="Default" />
+  <disable_collisions link1="franka2_fr3_hand" link2="franka2_fr3_leftfinger" reason="Adjacent" />
+  <disable_collisions link1="franka2_fr3_hand" link2="franka2_fr3_rightfinger" reason="Adjacent" />
+  <disable_collisions link1="table" link2="robot1_plate" reason="Adjacent" />
+  <disable_collisions link1="table" link2="robot2_plate" reason="Adjacent" />
+  <disable_collisions link1="franka1_fr3_link0" link2="robot1_plate" reason="Adjacent" />
+  <disable_collisions link1="franka2_fr3_link0" link2="robot2_plate" reason="Adjacent" />
+  <disable_collisions link1="franka1_fr3_link0" link2="table" reason="Never" />
+  <disable_collisions link1="franka2_fr3_link0" link2="table" reason="Never" />
+  <disable_collisions link1="franka1_fr3_link1" link2="table" reason="Never" />
+  <disable_collisions link1="franka2_fr3_link1" link2="table" reason="Never" />
+  <disable_collisions link1="franka1_fr3_link0" link2="franka2_fr3_link0" reason="Adjacent" />
 </robot>
