Commit message: MTC BUGS

File: src/franka_manipulation_env/srdf/bimanual_sim_srdf.xacro (robot description, xacro)
@@ -19,4 +19,22 @@
     <chain base_link="franka1_fr3_link0" tip_link="franka1_fr3_hand_tcp" />
   </group>
+  <group_state name="ready" group="franka1_arm">
+    <joint name="franka1_fr3_joint1" value="0" />
+    <joint name="franka1_fr3_joint2" value="${-pi/4}" />
+    <joint name="franka1_fr3_joint3" value="0" />
+    <joint name="franka1_fr3_joint4" value="${-3*pi/4}" />
+    <joint name="franka1_fr3_joint5" value="0" />
+    <joint name="franka1_fr3_joint6" value="${pi/2}" />
+    <joint name="franka1_fr3_joint7" value="${pi/4}" />
+  </group_state>
+  <group_state name="extended" group="franka1_arm">
+    <joint name="franka1_fr3_joint1" value="0" />
+    <joint name="franka1_fr3_joint2" value="0" />
+    <joint name="franka1_fr3_joint3" value="0" />
+    <joint name="franka1_fr3_joint4" value="-0.1" />
+    <joint name="franka1_fr3_joint5" value="0" />
+    <joint name="franka1_fr3_joint6" value="${pi/2}" />
+    <joint name="franka1_fr3_joint7" value="${pi/4}" />
+  </group_state>
   <group_state name="open" group="franka1_hand">
     <joint name="franka1_fr3_finger_joint1" value="0.035" />
@@ -44,4 +62,22 @@
     <chain base_link="franka2_fr3_link0" tip_link="franka2_fr3_hand_tcp" />
   </group>
+  <group_state name="ready" group="franka2_arm">
+    <joint name="franka2_fr3_joint1" value="0" />
+    <joint name="franka2_fr3_joint2" value="${-pi/4}" />
+    <joint name="franka2_fr3_joint3" value="0" />
+    <joint name="franka2_fr3_joint4" value="${-3*pi/4}" />
+    <joint name="franka2_fr3_joint5" value="0" />
+    <joint name="franka2_fr3_joint6" value="${pi/2}" />
+    <joint name="franka2_fr3_joint7" value="${pi/4}" />
+  </group_state>
+  <group_state name="extended" group="franka2_arm">
+    <joint name="franka2_fr3_joint1" value="0" />
+    <joint name="franka2_fr3_joint2" value="0" />
+    <joint name="franka2_fr3_joint3" value="0" />
+    <joint name="franka2_fr3_joint4" value="-0.1" />
+    <joint name="franka2_fr3_joint5" value="0" />
+    <joint name="franka2_fr3_joint6" value="${pi/2}" />
+    <joint name="franka2_fr3_joint7" value="${pi/4}" />
+  </group_state>
   <group name="bimanual_manipulator">
     <chain base_link="franka1_fr3_link0" tip_link="franka1_fr3_hand_tcp" />

File: src/franka_ros2/franka_fr3_moveit_config/srdf/group_definition.xacro (robot description, xacro)
@@ -3,23 +3,23 @@
   <xacro:macro name="group_definition" params="group_name arm_id tip_link">
     <group name="${group_name}">
-      <chain base_link="${arm_id}_link0" tip_link="${tip_link}"/>
+      <chain base_link="${arm_id}_link0" tip_link="${tip_link}" />
     </group>
     <group_state name="ready" group="${group_name}">
-      <joint name="${arm_id}_joint1" value="0"/>
-      <joint name="${arm_id}_joint2" value="${-pi/4}"/>
-      <joint name="${arm_id}_joint3" value="0"/>
-      <joint name="${arm_id}_joint4" value="${-3*pi/4}"/>
-      <joint name="${arm_id}_joint5" value="0"/>
-      <joint name="${arm_id}_joint6" value="${pi/2}"/>
-      <joint name="${arm_id}_joint7" value="${pi/4}"/>
+      <joint name="${arm_id}_joint1" value="0" />
+      <joint name="${arm_id}_joint2" value="${-pi/4}" />
+      <joint name="${arm_id}_joint3" value="0" />
+      <joint name="${arm_id}_joint4" value="${-3*pi/4}" />
+      <joint name="${arm_id}_joint5" value="0" />
+      <joint name="${arm_id}_joint6" value="${pi/2}" />
+      <joint name="${arm_id}_joint7" value="${pi/4}" />
     </group_state>
     <group_state name="extended" group="${group_name}">
-      <joint name="${arm_id}_joint1" value="0"/>
-      <joint name="${arm_id}_joint2" value="0"/>
-      <joint name="${arm_id}_joint3" value="0"/>
-      <joint name="${arm_id}_joint4" value="-0.1"/>
-      <joint name="${arm_id}_joint5" value="0"/>
-      <joint name="${arm_id}_joint6" value="${pi/2}"/>
-      <joint name="${arm_id}_joint7" value="${pi/4}"/>
+      <joint name="${arm_id}_joint1" value="0" />
+      <joint name="${arm_id}_joint2" value="0" />
+      <joint name="${arm_id}_joint3" value="0" />
+      <joint name="${arm_id}_joint4" value="-0.1" />
+      <joint name="${arm_id}_joint5" value="0" />
+      <joint name="${arm_id}_joint6" value="${pi/2}" />
+      <joint name="${arm_id}_joint7" value="${pi/4}" />
     </group_state>
   </xacro:macro>

Commit message: tf ready

File: src/franka_manipulation_env/srdf/bimanual_sim_srdf.xacro (robot description, xacro)
@@ -136,5 +136,4 @@
   <disable_collisions link1="franka1_fr3_link7" link2="franka1_fr3_rightfinger" reason="Never" />
   <disable_collisions link1="franka1_fr3_link8" link2="franka1_fr3_rightfinger" reason="Never" />
-  <disable_collisions link1="franka1_fr3_hand" link2="robot1_plate" reason="Never" />
   <disable_collisions link1="franka1_fr3_leftfinger" link2="franka1_fr3_rightfinger"
     reason="Default" />
@@ -178,13 +177,8 @@
   <disable_collisions link1="franka2_fr3_link7" link2="franka2_fr3_rightfinger" reason="Never" />
   <disable_collisions link1="franka2_fr3_link8" link2="franka2_fr3_rightfinger" reason="Never" />
-  <disable_collisions link1="franka2_fr3_hand" link2="robot2_plate" reason="Never" />
   <disable_collisions link1="franka2_fr3_leftfinger" link2="franka2_fr3_rightfinger"
     reason="Default" />
   <disable_collisions link1="franka2_fr3_hand" link2="franka2_fr3_leftfinger" reason="Adjacent" />
   <disable_collisions link1="franka2_fr3_hand" link2="franka2_fr3_rightfinger" reason="Adjacent" />
-  <disable_collisions link1="table" link2="robot1_plate" reason="Adjacent" />
-  <disable_collisions link1="table" link2="robot2_plate" reason="Adjacent" />
-  <disable_collisions link1="franka1_fr3_link0" link2="robot1_plate" reason="Adjacent" />
-  <disable_collisions link1="franka2_fr3_link0" link2="robot2_plate" reason="Adjacent" />
   <disable_collisions link1="franka1_fr3_link0" link2="table" reason="Never" />
   <disable_collisions link1="franka2_fr3_link0" link2="table" reason="Never" />

File: src/franka_manipulation_env/urdf/bimanual_custom.urdf.xacro (robot description, xacro)
@@ -2,9 +2,75 @@
 <robot xmlns:xacro="http://www.ros.org/wiki/xacro" name="idra_bimanual_setup">
   <xacro:include filename="$(find franka_description)/robots/common/franka_robot.xacro" />
+  <!-- Reference Frame Arguments -->
+  <xacro:arg name="table_x" default="0.0" />
+  <xacro:arg name="table_y" default="0.0" />
+  <xacro:arg name="table_z" default="0.2" />
+  <xacro:arg name="table_roll" default="0.0" />
+  <xacro:arg name="table_pitch" default="0.0" />
+  <xacro:arg name="table_yaw" default="0.0" />
+  <xacro:arg name="franka1_x" default="0.4375" />
+  <xacro:arg name="franka1_y" default="0.0" />
+  <xacro:arg name="franka1_z" default="0.06" />
+  <xacro:arg name="franka1_yaw" default="${pi}" />
+  <xacro:arg name="franka2_x" default="-0.4175" />
+  <xacro:arg name="franka2_y" default="0.0" />
+  <xacro:arg name="franka2_z" default="0.06" />
+  <xacro:arg name="franka2_yaw" default="0.0" />
+  <xacro:arg name="shared_x" default="0.4" />
+  <xacro:arg name="shared_y" default="0.0" />
+  <xacro:arg name="shared_z" default="0.05" />
+  <xacro:arg name="camera_x" default="0.6" />
+  <xacro:arg name="camera_y" default="1.0" />
+  <xacro:arg name="camera_z" default="1.3" />
+  <xacro:arg name="camera_roll" default="0.0" />
+  <xacro:arg name="camera_pitch" default="0.785" />
+  <xacro:arg name="camera_yaw" default="-1.57" />
+  <xacro:arg name="table_size_x" default="1.215" />
+  <xacro:arg name="table_size_y" default="0.6" />
+  <xacro:arg name="table_size_z" default="0.04" />
   <link name="world" />
   <joint name="world_joint" type="fixed">
-    <origin rpy="0 0 0" xyz="0 0 0.2" />
+    <origin rpy="$(arg table_roll) $(arg table_pitch) $(arg table_yaw)"
+            xyz="$(arg table_x) $(arg table_y) $(arg table_z)" />
     <parent link="world" />
     <child link="table" />
+  </joint>
+  <link name="shared_link">
+    <visual>
+      <geometry>
+        <sphere radius="0.02" />
+      </geometry>
+      <material name="shared_material">
+        <color rgba="0 1 0 0.5" />
+      </material>
+    </visual>
+  </link>
+  <joint name="table_to_shared" type="fixed">
+    <parent link="table" />
+    <child link="shared_link" />
+    <origin xyz="$(arg shared_x) $(arg shared_y) $(arg shared_z)" rpy="0 0 0" />
+  </joint>
+  <!-- AprilTag Fixed Reference -->
+  <link name="tag_0_fixed">
+    <visual>
+      <geometry>
+        <box size="0.05 0.05 0.001" />
+      </geometry>
+      <material name="tag_material">
+        <color rgba="0 0 0 1" />
+      </material>
+    </visual>
+  </link>
+  <joint name="table_to_tag_0" type="fixed">
+    <parent link="table" />
+    <child link="tag_0_fixed" />
+    <origin xyz="$(arg shared_x) $(arg shared_y) 0.0" rpy="0 0 0" />
+  </joint>
+  <link name="camera_link" />
+  <joint name="table_to_camera" type="fixed">
+    <parent link="table" />
+    <child link="camera_link" />
+    <origin xyz="$(arg camera_x) $(arg camera_y) $(arg camera_z)"
+            rpy="$(arg camera_roll) $(arg camera_pitch) $(arg camera_yaw)" />
   </joint>
   <material name="tablematerial">
@@ -17,43 +83,34 @@
     <visual>
       <geometry>
-        <box size="0.8 1.6 0.04" />
-      </geometry>
-      <origin xyz="0 0 -0.02" />
+        <box size="$(arg table_size_x) $(arg table_size_y) $(arg table_size_z)" />
+      </geometry>
+      <origin xyz="0 0 ${ -$(arg table_size_z) / 2 }" />
       <material name="tablematerial" />
     </visual>
+    <!-- Visual marker for table center -->
+    <visual>
+      <geometry>
+        <sphere radius="0.03" />
+      </geometry>
+      <material name="center_marker">
+        <color rgba="1 0 0 0.8" />
+      </material>
+    </visual>
     <collision>
       <geometry>
-        <box size="0.8 1.6 0.04" />
-      </geometry>
-      <origin xyz="0 0 -0.02" />
+        <box size="$(arg table_size_x) $(arg table_size_y) $(arg table_size_z)" />
+      </geometry>
+      <origin xyz="0 0 ${ -$(arg table_size_z) / 2 }" />
     </collision>
   </link>
-  <link name="robot1_plate">
-    <visual>
-      <geometry>
-        <box size="0.29 0.29 0.018" />
-      </geometry>
-      <origin xyz="0.145 0.145 0.009" />
-      <material name="platematerial" />
-    </visual>
-  </link>
-  <joint name="table_to_plate1" type="fixed">
-    <parent link="table" />
-    <child link="robot1_plate" />
-    <origin xyz="-0.2 0.6 0.0" />
-  </joint>
-  <link name="robot2_plate">
-    <visual>
-      <geometry>
-        <box size="0.29 0.29 0.018" />
-      </geometry>
-      <origin xyz="0.145 0.145 0.009" />
-      <material name="platematerial" />
-    </visual>
-  </link>
-  <joint name="table_to_plate2" type="fixed">
-    <parent link="table" />
-    <child link="robot2_plate" />
-    <origin xyz="-0.2 -0.6 0.0" />
+  <joint name="table_to_franka1" type="fixed">
+    <parent link="table" />
+    <child link="franka1_fr3_link0" />
+    <origin xyz="$(arg franka1_x) $(arg franka1_y) $(arg franka1_z)" rpy="0 0 $(arg franka1_yaw)" />
+  </joint>
+  <joint name="table_to_franka2" type="fixed">
+    <parent link="table" />
+    <child link="franka2_fr3_link0" />
+    <origin xyz="$(arg franka2_x) $(arg franka2_y) $(arg franka2_z)" rpy="0 0 $(arg franka2_yaw)" />
   </joint>
   <!-- Configuration Arguments -->
@@ -94,9 +151,4 @@
     rpy_ee="0 0 ${-pi/4}"
   />
-  <joint name="plate_to_franka1" type="fixed">
-    <parent link="robot1_plate" />
-    <child link="franka1_fr3_link0" />
-    <origin xyz="0.145 0.107 0.018" rpy="0 0 ${-pi/2}" />
-  </joint>
   <!-- Franka Robot 2 -->
   <xacro:franka_robot arm_id="fr3"
@@ -120,9 +172,4 @@
     rpy_ee="0 0 ${-pi/4}"
   />
-  <joint name="plate_to_franka2" type="fixed">
-    <parent link="robot2_plate" />
-    <child link="franka2_fr3_link0" />
-    <origin xyz="0.145 0.107 0.018" rpy="0 0 ${pi/2}" />
-  </joint>
   <!-- Hardware Interface Spawner -->
   <xacro:macro name="interface_spawner" params="robot_name">
